Commit message: refactor: Rename joint references and add additional parameters for hardware configuration

File: rh_p12_rn_a_description/ros2_control/rh_p12_rn_a.ros2_control.xacro (robot description, xacro)
@@ -38,5 +38,5 @@
         </hardware>
       </xacro:unless>
-      <joint name="${prefix}rh_r1_joint">
+      <joint name="${prefix}rh_r1">
         <command_interface name="position"/>
         <state_interface name="position"/>
@@ -46,5 +46,5 @@
       <xacro:if value="$(arg use_sim)">
         <joint name="${prefix}rh_r2">
-          <param name="mimic">${prefix}rh_r1_joint</param>
+          <param name="mimic">${prefix}rh_r1</param>
           <param name="multiplier">1</param>
           <state_interface name="position"/>
@@ -55,5 +55,5 @@
         </joint>
         <joint name="${prefix}rh_l1">
-          <param name="mimic">${prefix}rh_r1_joint</param>
+          <param name="mimic">${prefix}rh_r1</param>
           <param name="multiplier">1</param>
           <state_interface name="position"/>
@@ -64,5 +64,5 @@
         </joint>
         <joint name="${prefix}rh_l2">
-          <param name="mimic">${prefix}rh_r1_joint</param>
+          <param name="mimic">${prefix}rh_r1</param>
           <param name="multiplier">1</param>
           <state_interface name="position"/>
@@ -80,4 +80,9 @@
         <param name="type">dxl</param>
         <param name="ID">1</param>
+        <param name="Return Delay Time">0</param>
+        <param name="Min Position Limit">0</param>
+        <param name="Max Position Limit">740</param>
+        <param name="Profile Acceleration">0</param>
+        <param name="Profile Velocity">0</param>
       </gpio>
     </ros2_control>
