Commit message: refactor: Update joint references in configuration and description files

File: rh_p12_rn_a_description/gazebo/rh_p12_rn_a.gazebo.xacro (robot description, xacro)
@@ -29,5 +29,5 @@
   <xacro:Link reference="${prefix}rh_p12_rn_l1"/>
   <xacro:Link reference="${prefix}rh_p12_rn_l2"/>
-  <xacro:SimpleTransmission trans="${prefix}tran_r1" joint="${prefix}rh_r1_joint" actuator="${prefix}actuator1" />
+  <xacro:SimpleTransmission trans="${prefix}tran_r1" joint="${prefix}rh_r1" actuator="${prefix}actuator1" />
   <xacro:SimpleTransmission trans="${prefix}tran_r2" joint="${prefix}rh_r2" actuator="${prefix}actuator2" />
   <xacro:SimpleTransmission trans="${prefix}tran_l1" joint="${prefix}rh_l1" actuator="${prefix}actuator3" />

File: rh_p12_rn_a_description/urdf/rh_p12_rn_a.xacro (robot description, xacro)
@@ -102,5 +102,5 @@
       <limit velocity="6.5" effort="1000" lower="-0.001" upper="1.101" />
       <dynamics damping="0.7"/>
-      <mimic joint="${prefix}rh_r1_joint" multiplier="1"/>
+      <mimic joint="${prefix}rh_r1" multiplier="1"/>
     </joint>
     <!-- rh_p12_rn_l1 -->
@@ -135,5 +135,5 @@
       <limit velocity="6.5" effort="1000" lower="-0.001" upper="1.101" />
       <dynamics damping="0.7"/>
-      <mimic joint="${prefix}rh_r1_joint" multiplier="1"/>
+      <mimic joint="${prefix}rh_r1" multiplier="1"/>
     </joint>
     <!-- rh_p12_rn_l2 -->
